File: Hardware/KiCad7xx_UnoTypeC/KiCad7xx_UnoTypeC.kicad_sch (KiCad schematic)
At the start: 116 parts, among them T1 FDN340P, U1 MC33269ST, U2 LP2985-XXDBVR, U3 ATMEGA16U2-MU, U5 LMV358?MM, X1 POWERSUPPLY_DC21MMX, X2 USB-B_TH, Y1 16MHz, Y2 RESONATORMU

Commit message: feat: KiCad7xx_UnoTypeCにて既存のUnoRev3回路図をType-Cに変更
Parts:
- removed C11, C9: 22p, UNO-TH_Rev3e:C0603-ROUND, symbol UNO-TH_Rev3e-eagle-import:C-EU0603-RND
- removed FRAME1: A3-FRAME, UNO-TH_Rev3e:FRAME, symbol UNO-TH_Rev3e-eagle-import:A3-FRAME
- removed X2: USB-B_TH, UNO-TH_Rev3e:PN61729, symbol UNO-TH_Rev3e-eagle-import:PN61729
- removed Y1: 16MHz, UNO-TH_Rev3e:QS, symbol UNO-TH_Rev3e-eagle-import:XTAL/S
- added J1: USB_C_Receptacle_USB2.0, HRO_TYPE-C-31-M-12:HRO_TYPE-C-31-M-12, symbol Connector:USB_C_Receptacle_USB2.0
- added R3, R4: 5.1k, UNO-TH_Rev3e:R0603-ROUND, symbol Device:R
- added Y1: RESONATORMU, UNO-TH_Rev3e:RESONATOR, symbol UNO-TH_Rev3e-eagle-import:RESONATORMU
Connections:
- net D+: now also J1.A6 (D+), J1.B6 (D+)
- net D-: now also J1.A7 (D-), J1.B7 (D-)
- net GND: now also R3.1, R4.1, Y1.2
- net UGND: now also J1.A1 (GND), J1.A12 (GND), J1.B1 (GND), J1.B12 (GND)
- net USHIELD: now also J1.S1 (SHIELD)
- net XT1: now also Y1.3
- net XT2: now also Y1.1
- net XUSB: now also J1.A4 (VBUS), J1.A9 (VBUS), J1.B4 (VBUS), J1.B9 (VBUS)
- new net: J1.B5 (CC2), R4.2
- new net: J1.A5 (CC1), R3.2
- no-connect marks 0 -> 18
Other:
- moved on the sheet: AD0, C1, C10, C2, C3, C4, C5, C6, C7, C8, D1, D2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

Commit message: fix: HRO_TYPE-Cシンボルにて誤ったシンボルが選択されていた為、修正
Parts:
- J1: footprint HRO_TYPE-C-31-M-12:HRO_TYPE-C-31-M-12 -> Connector_USB:USB_C_Receptacle_HRO_TYPE-C-31-M-12
Changed lines of the file:
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@@
       (effects (font (size 1.27 1.27)))
     )
-    (property "Footprint" "HRO_TYPE-C-31-M-12:HRO_TYPE-C-31-M-12" (at 33.02 184.15 0)
+    (property "Footprint" "Connector_USB:USB_C_Receptacle_HRO_TYPE-C-31-M-12" (at 33.02 184.15 0)
       (effects (font (size 1.27 1.27)) hide)
     )
