File: Hardware/KiCad7xx_UNO-TH_Rev3e/KiCad7xx_UNO-TH_Rev3e.kicad_sch (KiCad schematic)
At the start: 116 parts, among them T1 FDN340P, U1 MC33269ST, U2 LP2985-XXDBVR, U3 ATMEGA16U2-MU, U5 LMV358?MM, X1 POWERSUPPLY_DC21MMX, X2 USB-B_TH, Y1 16MHz, Y2 RESONATORMU

Commit message: Add:Add converted to KiCad project
Parts:
- removed FRAME1: A3-FRAME, UNO-TH_Rev3e:FRAME, symbol UNO-TH_Rev3e-eagle-import:A3-FRAME
Connections:
- no-connect marks 0 -> 16
