File: Hardware/KiCad7xx_UNOSMD_V3/KiCad7xx_UNOSMD_V3.kicad_sch (KiCad schematic)
At the start: 72 parts, among them J1 -, J2 PINHD-1X18, T1 FDN340P, U1 MC33269ST, U2 LP2985-XXDBVR, U3 ATMEGA16U2, U4 ATMEGAXX8-MUR, U5 LMV358?MM, X1 POWERSUPPLY_DC21MMX, X2 USB-B_TH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

Commit message: Add:Add converted to KiCad project
Parts:
- removed FRAME1: DNP, UNOSMD_V3:FRAME, symbol UNOSMD_V3-eagle-import:A3-FRAME-STANDARD
Connections:
- no-connect marks 0 -> 18
