File: Hardware/KiCad7xx_UNOSMD_V3_TypeC_X301/KiCad7xx_UNOSMD_V3_TypeC_X301.kicad_pcb (KiCad board)
At the start: 2 copper layers, 68.6 x 53.3 mm, 76 parts, among them J1 -, J2 PINHD-1X18, J3 USB_C_Receptacle_USB2.0, T1 FDN340P, U1 MC33269ST, U2 LP2985-XXDBVR, U3 ATMEGA16U2, U4 ATMEGAXX8-MUR, U5 LMV358?MM, X1 POWERSUPPLY_DC21MMX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

Commit message: Add:X301の基板データに回路図の変更を追加
Parts:
- removed C11, C9: 22p, UNOSMD_V3:C0603-ROUND
- removed L0: YELLOW, UNOSMD_V3:CHIP-LED0805
- removed ON0: GREEN, UNOSMD_V3:CHIP-LED0805
- removed TP_CMP0, TP_GATE0, TP_LCMD0, TP_LL0, TP_ONL0: TP_SP, UNOSMD_V3:TP-SP
- added D4: CD1206-S01575, UNOSMD_V3:MINIMELF, F.Cu at (160.9, 123.9)
- added L3: YELLOW, UNOSMD_V3:CHIP-LED0805, F.Cu at (142.1, 89.5)
- added ON1: GREEN, UNOSMD_V3:CHIP-LED0805, F.Cu at (172.6, 95.1)
- added R5: 47k, Resistor_SMD:R_0603_1608Metric_Pad0.98x0.95mm_HandSolder, F.Cu at (129.3, 107.2)
- added TP_LCMD1: TP_SP, UNOSMD_V3:TP-SP, F.Cu at (133.1, 110.6)
- added TP_LL1: TP_SP, UNOSMD_V3:TP-SP, F.Cu at (139.7, 88.5)
- added TP_ONL1: TP_SP, UNOSMD_V3:TP-SP, F.Cu at (170.8, 96.6)
- added TP_USH0: TP_SP, UNOSMD_V3:TP-SP, F.Cu at (116.0, 94.6)
- added U6: BCM857BS, BCM857BS_SOT-363:SOT65P210X110-6N, F.Cu at (129.3, 104.8)
- J3: value USB_C_Receptacle_USB2.0 -> USB_C_Receptacle_USB2.0JAE_DX07S016JA1R1500
- Y1: value 16MHz -> RESONATORMU; footprint UNOSMD_V3:QS -> UNOSMD_V3:RESONATOR
- moved C2 3.01 mm to (129.3, 101.8), turned to 0 degrees
- moved Y1 1.83 mm to (134.8, 104.8)
- moved R1 0.45 mm to (133.7, 102.2)
Connections:
- J1 pad 8: VIN -> Net-(D4-PadA)
- RN1 pad 1: /CMP -> GND
- RN1 pad 2: /CMP -> unconnected-(RN1B-1-Pad2)
- RN1 pad 7: GND -> unconnected-(RN1B-2-Pad7)
- RN1 pad 8: VIN -> Net-(RN1A-2)
- T1 pad 3: /GATE_CMD -> Net-(T1-G)
- U5 pad 1: /GATE_CMD -> unconnected-(U5A-OUT-Pad1)
- U5 pad 2: +3V3 -> unconnected-(U5A--IN-Pad2)
- U5 pad 3: /CMP -> unconnected-(U5A-+IN-Pad3)
- Y1 pad 2: /XT1 -> GND
Routing:
- net VIN: track 82.6 -> 61.9 mm
- net Net-(RN1A-2): track 0.00 -> 19.5 mm, vias 0 -> 2
- net /GATE_CMD: track 19.2 -> 0.00 mm, vias 2 -> 0
- net /CMP: track 12.3 -> 0.00 mm, vias 1 -> 0
- net GND: track 24.2 -> 33.3 mm
- net +5V: track 229.2 -> 237.1 mm
- net Net-(T1-G): track 0.00 -> 7.14 mm
- net Net-(D4-PadA): track 0.00 -> 5.53 mm
- net +3V3: track 32.0 -> 27.4 mm
- net /USBVCC: track 21.3 -> 25.2 mm
- net /XT1: track 8.01 -> 6.04 mm
- net /XT2: track 8.13 -> 6.65 mm
