File: Hardware/KiCad7xx_UNOSMD_V3_TypeC_X302/KiCad7xx_UNOSMD_V3_TypeC_X302.kicad_sch (KiCad schematic)
At the start: 76 parts, among them J1 -, J2 PINHD-1X18, J3 USB_C_Receptacle_USB2.0JAE_DX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, T1 FDN340P, U1 MC33269ST, U2 LP2985-XXDBVR, U3 ATMEGA16U2, U4 ATMEGAXX8-MUR, U5 LMV358?MM, U6 BCM857BS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

Commit message: Add:MURからAUパッケージへ基板データを変更
Parts:
- U4: footprint UNOSMD_V3:MLF32 -> Package_QFP:TQFP-32_7x7mm_P0.8mm
Changed lines of the file:
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@@
       (effects (font (size 1.778 1.5113)) (justify left bottom))
     )
-    (property "Footprint" "UNOSMD_V3:MLF32" (at 266.7 170.18 0)
+    (property "Footprint" "Package_QFP:TQFP-32_7x7mm_P0.8mm" (at 266.7 170.18 0)
       (effects (font (size 1.27 1.27)) hide)
     )
